File: ALTIMETERS/TARS/TARS-MK1/TARS-MK1.kicad_pcb (KiCad board)
At the start: 2 copper layers, 127 x 257.8 mm, 99 parts, among them J11001 2309413-1, J3001 VENT_VALVE, J3002 BV_SERVO1, J3003 BV_SERVO2, J3004 PT1, J3005 PT2, J3006 PT3, J3007 UMBILLICAL, J5001 505575-0271, J5002 505575-0271, J5003 505575-0271, J5004 505575-0271, J5005 505575-0271, J5006 505575-0271, J6001 BATT1, J6002 BATT2_XT60, J6004 BATT4_CELL2, J6005 BATT4_CELL1, J6006 505575-0271, J6007 BATT5_CELL1, J6008 BATT3_JST, J6009 505575-0271, J7001 AC_SERVO1, J7002 AC_SERVO2, J7003 AC_SERVO3, Q3001 IRF540N, U1 RFM95W-915S2, U2001 Socket_BeagleBone_Black, U4001 Teensy4.1_bare, U5001 StratoLoggerCF, U5002 Telemetrum, U6001 D24V50F5, U6002 D36V28F3, U6003 LM7809_TO220, U6004 D36V50F6, U6005 D36V50F6, U6006 D24V50F5, U7001 LSM9DS1, U7002 KX122-1042, U7003 MS5611-01BA, U8001 ZOE-M8Q, U9001 Teensy4.1_bare, X1 SMACONNECTOR, X8001 SMACONNECTOR

Commit message: Added removed projects From ISS-PCB + Added .md's explaining folders
Other:
- net class Default removed
